File: kicad/ch2/ch2.kicad_sch (KiCad schematic)
At the start: 0 parts

Commit message: regular update
Other:
- added sheet CH02-KP2-07 (CH02-KP2-07.kicad_sch)
Changed lines of the file:
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@@
 	(paper "A4")
+	(sheet
+		(at 90.17 44.45)
+		(size 29.21 7.62)
+		(exclude_from_sim no)
+		(in_bom yes)
+		(on_board yes)
+		(dnp no)
+		(fields_autoplaced yes)
+		(stroke
+			(width 0.1524)
+			(type solid)
+		)
+		(fill
+			(color 0 0 0 0.0000)
+		)
+		(property "Sheetname" "CH02-KP2-07"
+			(at 90.17 43.7384 0)
+			(effects
+				(font
+					(size 1.27 1.27)
+				)
+				(justify left bottom)
+			)
+		)
+		(property "Sheetfile" "CH02-KP2-07.kicad_sch"
+			(at 90.17 52.6546 0)
+			(effects
+				(font
+					(size 1.27 1.27)
+				)
+				(justify left top)
+			)
+		)
+		(instances
+			(project "ch2"
+				(path "/fc72c8c5-f743-437f-8eef-093b2f91e0e9"
+					(page "3")
+				)
+			)
+		)
+	)
 	(sheet
 		(at 52.07 44.45)

Commit message: regular
Other:
- added sheet CH02-KP3-02 (CH02-KP3-02.kicad_sch)
- added sheet CH02-KP3-03 (CH02-KP3-03.kicad_sch)
- added sheet CH02-KP3-06 (CH02-KP3-06.kicad_sch)
- added sheet CH02-KP3-07 (CH02-KP3-07.kicad_sch)
- added sheet CH02-KP3-08 (CH02-KP3-08.kicad_sch)
- added sheet CH02-KP3-10 (CH02-KP3-10.kicad_sch)

Commit message: regular
Other:
- added sheet CH02-KP3-04 (CH02-KP3-04.kicad_sch)
- added sheet CH02-KP3-11 (CH02-KP3-11.kicad_sch)
- added sheet CH02-KP4-03 (CH2-KP4-03.kicad_sch)
- added sheet CH02-KP4-04 (CH2-KP4-04.kicad_sch)
- added sheet CH02-KP5-01 (CH2-KP5-01.kicad_sch)
- added sheet CH02-KP5-02 (CH02-KP5-02.kicad_sch)
- added sheet CH02-KP6-01 (CH02-KP6-01.kicad_sch)
